Commit message: Moved to robot_state_publisher added mpu imu

File: urdf/atrvjr.urdf.xacro (robot description, xacro)
@@ -51,10 +51,17 @@
       <child link="center_link"/>
   </joint>
-  <!-- Imu Link -->
-  <link name="imu_frame"/>
-  <joint name="base_imu_joint" type="fixed">
+  <!-- Crossbow Imu Link -->
+  <link name="cbimu_frame"/>
+  <joint name="base_cbimu_joint" type="fixed">
     <origin xyz="0 0 0.267" rpy="0 ${M_PI} 0"/>
     <parent link="center_link"/>
-    <child link="imu_frame"/>
+    <child link="cbimu_frame"/>
+  </joint>
+    <!-- MPU Imu Link -->
+  <link name="mpuimu_frame"/>
+  <joint name="base_mpuimu_joint" type="fixed">
+    <origin xyz="0 0 0.35" rpy="0 0 ${M_PI}"/>
+    <parent link="center_link"/>
+    <child link="mpuimu_frame"/>
   </joint>
 </robot>

Commit message: Added lrf frame, changed urdf to robot macro

File: urdf/atrvjr.urdf.xacro (robot description, xacro)
@@ -1,67 +1,128 @@
 <?xml version="1.0"?>
-<robot xmlns:xacro="http://www.ros.org/wiki/xacro" name="atrv">
-<!-- xacro parameters -->
-  <xacro:property name="M_PI" value="3.14159"/>
-  <!-- Robot parameters -->
-  <xacro:property name="ground_clearance" value="0.1525" />
-  <!-- This is not including the bumpers -->
-  <xacro:property name="chassis_length" value="0.64" />
-  <!-- This is including the bumpers -->
-  <xacro:property name="chassis_length_bumpers" value="0.78" />
-  <!-- This is not including the wheels -->
-  <xacro:property name="chassis_width" value="0.385" />
-  <!-- This is not including equipment and racks on the top -->
-  <xacro:property name="chassis_height" value="0.42" />
-<!-- xacro macros -->
-  <xacro:macro name="default_inertial" params="mass">
-    <inertial>
-      <mass value="${mass}" />
-      <inertia ixx="1.0" ixy="0.0" ixz="0.0"
-               iyy="1.0" iyz="0.0"
-               izz="1.0" />
-      </inertial>
-  </xacro:macro>
-<!-- links -->
-  <!-- base_link -->
-  <!-- The frame of the floor directly below the center_link and -->
-  <!-- is needed for the navigation stack to work properly -->
-  <link name="base_link"></link>
-  <!-- center_link -->
-  <!-- The link that is the origin of all of the components of the -->
-  <!-- robot and should also represent the main chassis via inertial, -->
-  <!-- visual, and geometry elements of the link -->
-  <link name="center_link">
-    <xacro:default_inertial mass="50"/>
-    <visual>
-      <geometry>
-        <mesh filename="package://atrvjr_description/meshes/atrvjr_chassis_v5.dae"/>
-      </geometry>
-    </visual>
-    <collision>
-      <origin xyz="0 0 ${chassis_height/2.0}" rpy="0 0 0" />
-      <geometry>
-        <box size="${chassis_length} ${chassis_width} ${chassis_height}" />
-      </geometry>
-    </collision>
-  </link>
-  <!-- base_link -> center_link -->
-  <joint name="base_link_joint" type="fixed">
-      <origin xyz="0 0 ${ground_clearance}" rpy="0 0 0"/>
-      <parent link="base_link"/>
-      <child link="center_link"/>
-  </joint>
-  <!-- Crossbow Imu Link -->
-  <link name="cbimu_frame"/>
-  <joint name="base_cbimu_joint" type="fixed">
-    <origin xyz="0 0 0.267" rpy="0 ${M_PI} 0"/>
-    <parent link="center_link"/>
-    <child link="cbimu_frame"/>
-  </joint>
-    <!-- MPU Imu Link -->
-  <link name="mpuimu_frame"/>
-  <joint name="base_mpuimu_joint" type="fixed">
-    <origin xyz="0 0 0.35" rpy="0 0 ${M_PI}"/>
-    <parent link="center_link"/>
-    <child link="mpuimu_frame"/>
-  </joint>
+<robot xmlns:xacro="http://www.ros.org/wiki/xacro" name="atrvjr_ur5">
+    <xacro:macro name="atrvjr" params="armConnectionFrame">
+    <!-- xacro parameters -->
+    <xacro:property name="M_PI" value="3.14159"/>
+    <!-- Robot parameters -->
+    <xacro:property name="center_height" value="0.1525" />
+    <!-- This is not including the bumpers -->
+    <xacro:property name="chassis_length" value="0.64" />
+    <!-- This is including the bumpers -->
+    <xacro:property name="chassis_length_bumpers" value="0.78" />
+    <!-- This is not including the wheels -->
+    <xacro:property name="chassis_width" value="0.385" />
+    <!-- This is not including equipment and racks on the top -->
+    <xacro:property name="chassis_height" value="0.42" />
+    <!-- Wheel properties -->
+    <xacro:property name="wheel_radius" value="0.155"/>
+    <xacro:property name="wheel_width" value="0.095"/>
+    <xacro:property name="wheel_base" value="0.38"/> <!-- aka distance between axis -->
+    <!-- xacro macros -->
+    <xacro:macro name="default_inertial" params="mass">
+        <inertial>
+        <mass value="${mass}" />
+        <inertia ixx="1.0" ixy="0.0" ixz="0.0"
+                iyy="1.0" iyz="0.0"
+                izz="1.0" />
+        </inertial>
+    </xacro:macro>
+    <xacro:macro name="wheel" params="prefix reflect_x reflect_y">
+        <link name="${prefix}_wheel_link">
+            <xacro:default_inertial mass="1"/>
+            <collision>
+                <origin xyz="0 0 ${wheel_width/2}" rpy="0 0 0" />
+                <geometry>
+                    <cylinder radius="${wheel_radius}" length="${wheel_width}"/>
+                </geometry>
+            </collision>
+        </link>
+        <!-- base_link -> ${prefix}_wheel_link -->
+        <joint name="${prefix}_wheel_joint" type="fixed">
+            <parent link="center_link"/>
+            <child link="${prefix}_wheel_link"/>
+            <origin xyz="${(wheel_base/2)*reflect_x} ${(chassis_width/2 + 0.02)*reflect_y} 0"
+            rpy="${(M_PI/2)*reflect_y*-1} 0 0"/>
+        </joint>
+    </xacro:macro>
+    <!-- left_front_wheel_link -->
+    <xacro:wheel prefix="left_front" reflect_x="1" reflect_y="1" />
+    <!-- left_rear_wheel_link -->
+    <xacro:wheel prefix="left_rear" reflect_x="-1" reflect_y="1" />
+    <!-- right_front_wheel_link -->
+    <xacro:wheel prefix="right_front" reflect_x="1" reflect_y="-1" />
+    <!-- right_rear_wheel_link -->
+    <xacro:wheel prefix="right_rear" reflect_x="-1" reflect_y="-1" />
+    <!-- links -->
+    <!-- base_link -->
+    <!-- The frame of the floor directly below the center_link and -->
+    <!-- is needed for the navigation stack to work properly -->
+    <link name="base_link"></link>
+    <!-- center_link -->
+    <!-- The link that is the origin of all of the components of the -->
+    <!-- robot and should also represent the main chassis via inertial, -->
+    <!-- visual, and geometry elements of the link -->
+    <link name="center_link">
+        <xacro:default_inertial mass="50"/>
+        <visual>
+            <geometry>
+                <mesh filename="package://atrvjr_description/meshes/atrvjr_chassis_v5.dae"/>
+            </geometry>
+        </visual>
+        <collision>
+            <origin xyz="0 0 ${chassis_height/2.0 - 0.10}" rpy="0 0 0" />
+            <geometry>
+                <box size="${chassis_length} ${chassis_width} ${chassis_height}" />
+            </geometry>
+        </collision>
+    </link>
+    <!-- base_link -> center_link -->
+    <joint name="base_link_joint" type="fixed">
+        <origin xyz="0 0 ${center_height}" rpy="0 0 0"/>
+        <parent link="base_link"/>
+        <child link="center_link"/>
+    </joint>
+    <!-- Crossbow Imu Link -->
+    <link name="cbimu_frame"/>
+    <joint name="base_cbimu_joint" type="fixed">
+        <origin xyz="0 0 0.267" rpy="0 ${M_PI} 0"/>
+        <parent link="center_link"/>
+        <child link="cbimu_frame"/>
+    </joint>
+        <!-- MPU Imu Link -->
+    <link name="mpuimu_frame"/>
+    <joint name="base_mpuimu_joint" type="fixed">
+        <origin xyz="0 0 0.35" rpy="0 0 ${M_PI}"/>
+        <parent link="center_link"/>
+        <child link="mpuimu_frame"/>
+    </joint>
+    <!-- Arm Link -->
+    <link name="${armConnectionFrame}"/>
+    <joint name="$to_{armConnectionFrame}_joint" type="fixed">
+        <origin xyz="0 0 0.40" rpy="0 0 0"/>
+        <parent link="center_link"/>
+        <child link="${armConnectionFrame}"/>
+    </joint>
+    <!-- Hokuyo Link -->
+    <link name="lrf_frame"/>
+    <joint name="lrf_joint" type="fixed">
+        <origin xyz="0.2 0 0.35" rpy="0 0 0"/>
+        <parent link="center_link"/>
+        <child link="lrf_frame"/>
+    </joint>
+    </xacro:macro>
+    <xacro:macro name="ur5" params="baseframe">
+        <!-- common stuff -->
+        <xacro:include filename="$(find ur_description)/urdf/common.gazebo.xacro" />
+        <!-- ur5 -->
+        <xacro:include filename="$(find ur_description)/urdf/ur5.urdf.xacro" />
+        <!-- arm -->
+        <xacro:ur5_robot prefix="ur5_" joint_limited="false"/>
+        <joint name="$from_{baseframe}_joint" type="fixed">
+            <parent link="${baseframe}" />
+            <child link = "ur5_base_link" />
+            <origin xyz="0.0 0.0 0.0" rpy="0.0 0.0 0.0" />
+        </joint>
+    </xacro:macro>
+    <xacro:atrvjr armConnectionFrame="arm_base_frame" />
+    <!--<xacro:ur5 baseframe="arm_base_frame" />-->
 </robot>

Commit message: Fixed mpu orientation, added novatel frame

File: urdf/atrvjr.urdf.xacro (robot description, xacro)
@@ -92,5 +92,5 @@
     <link name="mpuimu_frame"/>
     <joint name="base_mpuimu_joint" type="fixed">
-        <origin xyz="0 0 0.35" rpy="0 0 ${M_PI}"/>
+        <origin xyz="0 0 0.35" rpy="0 0 ${M_PI/2.0}"/>
         <parent link="center_link"/>
         <child link="mpuimu_frame"/>
@@ -109,4 +109,11 @@
         <parent link="center_link"/>
         <child link="lrf_frame"/>
+    </joint>
+    <!-- Hokuyo Link -->
+    <link name="novatel"/>
+    <joint name="novatel_joint" type="fixed">
+        <origin xyz="-0.15 0.1 0.4" rpy="0 0 0"/>
+        <parent link="center_link"/>
+        <child link="novatel"/>
     </joint>
     </xacro:macro>

Commit message: Clean up, added ATRV-Jr and UR5 launch file

File: urdf/atrvjr.urdf.xacro (robot description, xacro)
@@ -1,135 +1,5 @@
 <?xml version="1.0"?>
-<robot xmlns:xacro="http://www.ros.org/wiki/xacro" name="atrvjr_ur5">
-    <xacro:macro name="atrvjr" params="armConnectionFrame">
-    <!-- xacro parameters -->
-    <xacro:property name="M_PI" value="3.14159"/>
-    <!-- Robot parameters -->
-    <xacro:property name="center_height" value="0.1525" />
-    <!-- This is not including the bumpers -->
-    <xacro:property name="chassis_length" value="0.64" />
-    <!-- This is including the bumpers -->
-    <xacro:property name="chassis_length_bumpers" value="0.78" />
-    <!-- This is not including the wheels -->
-    <xacro:property name="chassis_width" value="0.385" />
-    <!-- This is not including equipment and racks on the top -->
-    <xacro:property name="chassis_height" value="0.42" />
-    <!-- Wheel properties -->
-    <xacro:property name="wheel_radius" value="0.155"/>
-    <xacro:property name="wheel_width" value="0.095"/>
-    <xacro:property name="wheel_base" value="0.38"/> <!-- aka distance between axis -->
-    <!-- xacro macros -->
-    <xacro:macro name="default_inertial" params="mass">
-        <inertial>
-        <mass value="${mass}" />
-        <inertia ixx="1.0" ixy="0.0" ixz="0.0"
-                iyy="1.0" iyz="0.0"
-                izz="1.0" />
-        </inertial>
-    </xacro:macro>
-    <xacro:macro name="wheel" params="prefix reflect_x reflect_y">
-        <link name="${prefix}_wheel_link">
-            <xacro:default_inertial mass="1"/>
-            <collision>
-                <origin xyz="0 0 ${wheel_width/2}" rpy="0 0 0" />
-                <geometry>
-                    <cylinder radius="${wheel_radius}" length="${wheel_width}"/>
-                </geometry>
-            </collision>
-        </link>
-        <!-- base_link -> ${prefix}_wheel_link -->
-        <joint name="${prefix}_wheel_joint" type="fixed">
-            <parent link="center_link"/>
-            <child link="${prefix}_wheel_link"/>
-            <origin xyz="${(wheel_base/2)*reflect_x} ${(chassis_width/2 + 0.02)*reflect_y} 0"
-            rpy="${(M_PI/2)*reflect_y*-1} 0 0"/>
-        </joint>
-    </xacro:macro>
-    <!-- left_front_wheel_link -->
-    <xacro:wheel prefix="left_front" reflect_x="1" reflect_y="1" />
-    <!-- left_rear_wheel_link -->
-    <xacro:wheel prefix="left_rear" reflect_x="-1" reflect_y="1" />
-    <!-- right_front_wheel_link -->
-    <xacro:wheel prefix="right_front" reflect_x="1" reflect_y="-1" />
-    <!-- right_rear_wheel_link -->
-    <xacro:wheel prefix="right_rear" reflect_x="-1" reflect_y="-1" />
-    <!-- links -->
-    <!-- base_link -->
-    <!-- The frame of the floor directly below the center_link and -->
-    <!-- is needed for the navigation stack to work properly -->
-    <link name="base_link"></link>
-    <!-- center_link -->
-    <!-- The link that is the origin of all of the components of the -->
-    <!-- robot and should also represent the main chassis via inertial, -->
-    <!-- visual, and geometry elements of the link -->
-    <link name="center_link">
-        <xacro:default_inertial mass="50"/>
-        <visual>
-            <geometry>
-                <mesh filename="package://atrvjr_description/meshes/atrvjr_chassis_v5.dae"/>
-            </geometry>
-        </visual>
-        <collision>
-            <origin xyz="0 0 ${chassis_height/2.0 - 0.10}" rpy="0 0 0" />
-            <geometry>
-                <box size="${chassis_length} ${chassis_width} ${chassis_height}" />
-            </geometry>
-        </collision>
-    </link>
-    <!-- base_link -> center_link -->
-    <joint name="base_link_joint" type="fixed">
-        <origin xyz="0 0 ${center_height}" rpy="0 0 0"/>
-        <parent link="base_link"/>
-        <child link="center_link"/>
-    </joint>
-    <!-- Crossbow Imu Link -->
-    <link name="cbimu_frame"/>
-    <joint name="base_cbimu_joint" type="fixed">
-        <origin xyz="0 0 0.267" rpy="0 ${M_PI} 0"/>
-        <parent link="center_link"/>
-        <child link="cbimu_frame"/>
-    </joint>
-        <!-- MPU Imu Link -->
-    <link name="mpuimu_frame"/>
-    <joint name="base_mpuimu_joint" type="fixed">
-        <origin xyz="0 0 0.35" rpy="0 0 ${M_PI/2.0}"/>
-        <parent link="center_link"/>
-        <child link="mpuimu_frame"/>
-    </joint>
-    <!-- Arm Link -->
-    <link name="${armConnectionFrame}"/>
-    <joint name="$to_{armConnectionFrame}_joint" type="fixed">
-        <origin xyz="0 0 0.40" rpy="0 0 0"/>
-        <parent link="center_link"/>
-        <child link="${armConnectionFrame}"/>
-    </joint>
-    <!-- Hokuyo Link -->
-    <link name="lrf_frame"/>
-    <joint name="lrf_joint" type="fixed">
-        <origin xyz="0.2 0 0.35" rpy="0 0 0"/>
-        <parent link="center_link"/>
-        <child link="lrf_frame"/>
-    </joint>
-    <!-- Hokuyo Link -->
-    <link name="novatel"/>
-    <joint name="novatel_joint" type="fixed">
-        <origin xyz="-0.15 0.1 0.4" rpy="0 0 0"/>
-        <parent link="center_link"/>
-        <child link="novatel"/>
-    </joint>
-    </xacro:macro>
-    <xacro:macro name="ur5" params="baseframe">
-        <!-- common stuff -->
-        <xacro:include filename="$(find ur_description)/urdf/common.gazebo.xacro" />
-        <!-- ur5 -->
-        <xacro:include filename="$(find ur_description)/urdf/ur5.urdf.xacro" />
-        <!-- arm -->
-        <xacro:ur5_robot prefix="ur5_" joint_limited="false"/>
-        <joint name="$from_{baseframe}_joint" type="fixed">
-            <parent link="${baseframe}" />
-            <child link = "ur5_base_link" />
-            <origin xyz="0.0 0.0 0.0" rpy="0.0 0.0 0.0" />
-        </joint>
-    </xacro:macro>
-    <xacro:atrvjr armConnectionFrame="arm_base_frame" />
-    <!--<xacro:ur5 baseframe="arm_base_frame" />-->
+<robot xmlns:xacro="http://www.ros.org/wiki/xacro" name="atrvjr">
+  <xacro:include filename="$(find atrvjr_description)/urdf/atrvjr.xacro" />
+  <xacro:atrvjr armConnectionFrame="arm_base_frame" />
 </robot>
